File: JP280C1.kicad_pcb (KiCad board)
At the start: 2 copper layers, 110 x 44 mm, 13 parts, among them J1 Ribbon Cable (C)

Commit message: completed wiring
Parts:
- moved SK1 20.5 mm to (49.5, 172.7)
- moved J1 16.7 mm to (109.2, 172.7)
- moved SK2 16.7 mm to (39.4, 172.7)
- moved SK3 15.5 mm to (78.7, 172.7)
- moved SK4 14.2 mm to (68.6, 172.7)
- moved R3 14.0 mm to (34.3, 166.4)
- moved R1 11.5 mm to (50.8, 167.6)
- moved R4 10.2 mm to (38.1, 162.6)
- moved R2 8.98 mm to (53.3, 163.8)
- moved SK5 2.00 mm to (72.0, 139.7)
- moved SK6 2.00 mm to (45.0, 139.7)
- moved SK7 2.00 mm to (99.0, 139.7)
- moved SK8 2.00 mm to (126.0, 139.7)
Routing:
- net GND: track 0.00 -> 214.8 mm
- net Net-(J1-Pad5): track 0.00 -> 86.0 mm
- net Net-(J1-Pad9): track 0.00 -> 82.8 mm
- net Net-(J1-Pad6): track 0.00 -> 69.7 mm, vias 0 -> 2
- net Net-(J1-Pad10): track 0.00 -> 57.6 mm
- net Net-(J1-Pad8): track 0.00 -> 45.1 mm
- net Net-(J1-Pad7): track 0.00 -> 41.6 mm
- net Net-(J1-Pad3): track 0.00 -> 35.1 mm
- net Net-(J1-Pad4): track 0.00 -> 25.0 mm
- net Net-(J1-Pad1): track 0.00 -> 23.9 mm
- net Net-(R1-Pad2): track 0.00 -> 18.1 mm
- net Net-(R3-Pad2): track 0.00 -> 15.8 mm
- net Net-(J1-Pad2): track 0.00 -> 13.8 mm
