File: JP280C1.kicad_pcb (KiCad board)
At the start: 2 copper layers, 110 x 44 mm, 13 parts, among them J1 Ribbon Cable (C)

Commit message: corrected placement of SK7 and SK8
Parts:
- moved SK7 27.0 mm to (126.0, 139.7)
- moved SK8 27.0 mm to (99.0, 139.7)
Routing:
- net GND: track 214.8 -> 160.8 mm
- net Net-(J1-Pad7): track 41.6 -> 80.1 mm
- net Net-(J1-Pad8): track 45.1 -> 36.2 mm

Commit message: preparing to add libs as submodule
Routing:
- net GND: track 160.8 -> 214.8 mm

Commit message: added copper fill
Parts:
- added R0: 0R, TAC:Wire_Bridge_P7.62mm_Horizontal, F.Cu at (90.2, 163.8)
Connections:
- R1 pad 1: Net-(J1-Pad6) -> Net-(R0-Pad1)
- SK1 pad 2: Net-(J1-Pad6) -> Net-(R0-Pad1)
Routing:
- net Net-(J1-Pad6): track 69.7 -> 9.42 mm, vias 2 -> 0
- net Net-(R0-Pad1): track 0.00 -> 52.7 mm
Other:
- board text added: "JP280C1"
- board text added: "v1.0"

Commit message: schematic done for JP280C2
Routing:
- net Net-(J1-Pad8): track 36.2 -> 60.9 mm

Commit message: narrowed JP208C1 to 107 mm; added engravings to Cmts.User layer
Other:
- board size 110 x 44 mm -> 107 x 44 mm
